Commit message: updated

File: install/arduinobot_description/share/arduinobot_description/urdf/arduinobot.urdf.xacro (robot description, xacro)
@@ -19,4 +19,12 @@
       <material name="blue"/>
     </visual>
+    <collision>
+      <geometry>
+        <sphere radius="0.2"/>
+      </geometry>
+    </collision>
+    <xacro:inertial_cylinder mass="5" length="0.6" radius="0.2">
+            <origin xyz="0 0 0" rpy="0 0 0"/>
+    </xacro:inertial_cylinder>
   </link>
   <link name="head">
@@ -27,4 +35,12 @@
       <material name="white"/>
     </visual>
+    <collision>
+      <geometry>
+        <sphere radius="0.2"/>
+      </geometry>
+    </collision>
+    <xacro:inertial_sphere mass="5" radius="0.2">
+            <origin xyz="0 0 0" rpy="0 0 0"/>
+    </xacro:inertial_sphere>
   </link>
   <joint name="head_swivel" type="continuous">

Commit message: updated

File: install/arduinobot_description/share/arduinobot_description/urdf/arduinobot.urdf.xacro (robot description, xacro)
@@ -24,7 +24,4 @@
       </geometry>
     </collision>
-    <xacro:inertial_cylinder mass="5" length="0.6" radius="0.2">
-            <origin xyz="0 0 0" rpy="0 0 0"/>
-    </xacro:inertial_cylinder>
   </link>
   <link name="head">
